File: Particle-Gateway.brd (EAGLE design)
At the start: 47 x 40.6 mm, 27 parts, among them J2 GROVE-I2C, J3 Lipo Battery, J4 GROVE-I2C, J5 CON_HEADER_1X08-PTH, P1 PADSMALL, U1 AMS1117-3.3

Commit message: Connect DIO2 to D3
Connections:
- net D3: now also U$3.DIO2
Routing:
- net D3: track 2.73 -> 25.7 mm, vias 0 -> 2
Changed lines of the file:
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@@
 <?xml version="1.0" encoding="utf-8"?>
 <!DOCTYPE eagle SYSTEM "eagle.dtd">
-<eagle version="7.3.0">
+<eagle version="7.4.0">
 <drawing>
 <settings>
@@
 <setting verticaltext="up"/>
 </settings>
-<grid distance="50" unitdist="mil" unit="mil" style="lines" multiple="1" display="yes" altdistance="5" altunitdist="mil" altunit="mil"/>
+<grid distance="25" unitdist="mil" unit="mil" style="lines" multiple="1" display="yes" altdistance="5" altunitdist="mil" altunit="mil"/>
 <layers>
 <layer number="1" name="Top" color="4" fill="1" visible="yes" active="yes"/>
@@
 <wire x1="17.98" y1="8.817" x2="17.98" y2="11.33" width="0.8128" layer="1"/>
 <wire x1="17.98" y1="8.817" x2="18.00225" y2="8.60425" width="0.4064" layer="1"/>
+<contactref element="U$3" pad="DIO2"/>
+<wire x1="32.074" y1="21.2052" x2="31.75" y2="21.2052" width="0.4064" layer="16"/>
+<wire x1="31.75" y1="21.2052" x2="31.75" y2="19.685" width="0.4064" layer="16"/>
+<wire x1="31.75" y1="19.685" x2="28.575" y2="16.51" width="0.4064" layer="16"/>
+<wire x1="28.575" y1="16.51" x2="28.575" y2="14.605" width="0.4064" layer="16"/>
+<via x="28.575" y="14.605" extent="1-16" drill="0.6" shape="square"/>
+<wire x1="28.575" y1="14.605" x2="17.78" y2="15.24" width="0.4064" layer="1"/>
+<via x="17.78" y="15.24" extent="1-16" drill="0.6" shape="square"/>
+<wire x1="17.78" y1="15.24" x2="17.98" y2="11.33" width="0.4064" layer="16"/>
 </signal>
 <signal name="D2">
